File: Arduino Project/Arduino Project.sch (KiCad schematic (older format))
At the start: 21 parts, among them U1 Teensy3.5

Commit message: Final sch ready for review
Parts:
- removed U?: TXB0108DQSR, Package_SON:USON-20_2x4mm_P0.4mm, symbol Logic_LevelTranslator:TXB0108DQSR
- added PWM-?: Conn_01x03, symbol Connector_Generic:Conn_01x03
Connections:
- net labels removed: LED_PWM
- no-connect marks 42 -> 77
Other:
- moved on the sheet: XT-60
Changed lines of the file:
@@
 L Connector_Generic:Conn_01x02 XT-60
 U 1 1 5D95EA1A
-P 6900 1250
-F 0 "XT-60" H 6980 1242 50  0000 L CNN
-F 1 "Conn_01x02" H 6980 1151 50  0000 L CNN
-F 2 "" H 6900 1250 50  0001 C CNN
-F 3 "~" H 6900 1250 50  0001 C CNN
-	1    6900 1250
+P 7500 1250
+F 0 "XT-60" H 7580 1242 50  0000 L CNN
+F 1 "Conn_01x02" H 7580 1151 50  0000 L CNN
+F 2 "" H 7500 1250 50  0001 C CNN
+F 3 "~" H 7500 1250 50  0001 C CNN
+	1    7500 1250
 	1    0    0    -1
 $EndComp
@@
 L power:GND #PWR?
 U 1 1 5D9602AD
-P 6700 1350
-F 0 "#PWR?" H 6700 1100 50  0001 C CNN
-F 1 "GND" V 6705 1222 50  0000 R CNN
-F 2 "" H 6700 1350 50  0001 C CNN
-F 3 "" H 6700 1350 50  0001 C CNN
-	1    6700 1350
+P 7300 1350
+F 0 "#PWR?" H 7300 1100 50  0001 C CNN
+F 1 "GND" V 7305 1222 50  0000 R CNN
+F 2 "" H 7300 1350 50  0001 C CNN
+F 3 "" H 7300 1350 50  0001 C CNN
+	1    7300 1350
 	0    1    1    0
 $EndComp
@@
 L power:+5V #PWR?
 U 1 1 5D95FEAE
-P 6700 1250
-F 0 "#PWR?" H 6700 1100 50  0001 C CNN
-F 1 "+5V" V 6715 1378 50  0000 L CNN
-F 2 "" H 6700 1250 50  0001 C CNN
-F 3 "" H 6700 1250 50  0001 C CNN
-	1    6700 1250
+P 7300 1250
+F 0 "#PWR?" H 7300 1100 50  0001 C CNN
+F 1 "+5V" V 7315 1378 50  0000 L CNN
+F 2 "" H 7300 1250 50  0001 C CNN
+F 3 "" H 7300 1250 50  0001 C CNN
+	1    7300 1250
 	0    -1   -1   0
 $EndComp
@@
 Text GLabel 1150 5100 0    50   Input ~ 0
 PWM_12
-Text GLabel 5700 6050 1    50   Input ~ 0
-PWM_14
 $Comp
 L power:+3.3V #PWR?
@@
 NoConn ~ 3450 3700
 NoConn ~ 3450 3800
-$Comp
-L Logic_LevelTranslator:TXB0108DQSR U?
-U 1 1 5D97383B
-P 5400 6450
-F 0 "U?" V 5150 5700 50  0000 R CNN
-F 1 "TXB0108DQSR" V 5650 5700 50  0000 R CNN
-F 2 "Package_SON:USON-20_2x4mm_P0.4mm" H 5400 5700 50  0001 C CNN
-F 3 "http://www.ti.com/lit/ds/symlink/txb0108.pdf" H 5400 6350 50  0001 C CNN
-	1    5400 6450
-	0    1    1    0
-$EndComp
-$Comp
-L power:GND #PWR?
-U 1 1 5D9745E7
-P 4700 6450
-F 0 "#PWR?" H 4700 6200 50  0001 C CNN
-F 1 "GND" V 4705 6322 50  0000 R CNN
-F 2 "" H 4700 6450 50  0001 C CNN
-F 3 "" H 4700 6450 50  0001 C CNN
-	1    4700 6450
-	0    1    1    0
-$EndComp
-$Comp
-L power:+3.3V #PWR?
-U 1 1 5D97491A
-P 6100 6350
-F 0 "#PWR?" H 6100 6200 50  0001 C CNN
-F 1 "+3.3V" V 6115 6478 50  0000 L CNN
-F 2 "" H 6100 6350 50  0001 C CNN
-F 3 "" H 6100 6350 50  0001 C CNN
-	1    6100 6350
-	0    1    1    0
-$EndComp
+Text GLabel 9750 4800 0    50   Input ~ 0
+PWM_14
+$Comp
+L Connector_Generic:Conn_01x03 PWM-?
+U 1 1 5D97065B
+P 9950 4900
+F 0 "PWM-?" H 10030 4942 50  0000 L CNN
+F 1 "Conn_01x03" H 10030 4851 50  0000 L CNN
+F 2 "" H 9950 4900 50  0001 C CNN
+F 3 "~" H 9950 4900 50  0001 C CNN
+	1    9950 4900
+	1    0    0    -1
+$EndComp
+$Comp
+L power:GND #PWR?
+U 1 1 5D9706AF
+P 9750 5000
+F 0 "#PWR?" H 9750 4750 50  0001 C CNN
+F 1 "GND" V 9755 4872 50  0000 R CNN
+F 2 "" H 9750 5000 50  0001 C CNN
+F 3 "" H 9750 5000 50  0001 C CNN
+	1    9750 5000
+	0    1    1    0
+$EndComp
+NoConn ~ 9750 4900
+NoConn ~ 3450 5000
+NoConn ~ 3450 4900
+NoConn ~ 3450 4500
+NoConn ~ 3450 4400
+NoConn ~ 3450 4300
+NoConn ~ 3450 4200
 $Comp
 L power:+5V #PWR?
-U 1 1 5D974989
-P 6100 6550
-F 0 "#PWR?" H 6100 6400 50  0001 C CNN
-F 1 "+5V" V 6115 6678 50  0000 L CNN
-F 2 "" H 6100 6550 50  0001 C CNN
-F 3 "" H 6100 6550 50  0001 C CNN
-	1    6100 6550
-	0    1    1    0
-$EndComp
-Text GLabel 5700 6850 3    50   Input ~ 0
-LED_PWM
+U 1 1 5D971052
+P 1150 3600
+F 0 "#PWR?" H 1150 3450 50  0001 C CNN
+F 1 "+5V" V 1165 3728 50  0000 L CNN
+F 2 "" H 1150 3600 50  0001 C CNN
+F 3 "" H 1150 3600 50  0001 C CNN
+	1    1150 3600
+	0    -1   -1   0
+$EndComp
+NoConn ~ 3450 4700
+NoConn ~ 1150 1100
+NoConn ~ 1150 1200
+NoConn ~ 1150 1300
+NoConn ~ 1150 1800
+NoConn ~ 1150 1900
+NoConn ~ 1150 2000
+NoConn ~ 1150 2300
+NoConn ~ 1150 2400
+NoConn ~ 1150 2500
+NoConn ~ 1150 2600
+NoConn ~ 1150 2700
+NoConn ~ 1150 2800
+NoConn ~ 1150 2900
+NoConn ~ 1150 3000
+NoConn ~ 1150 3300
+NoConn ~ 1150 3400
+NoConn ~ 1150 3500
+NoConn ~ 1150 3800
+NoConn ~ 1150 3900
+NoConn ~ 1150 4000
+NoConn ~ 1150 4100
+NoConn ~ 1150 4600
+NoConn ~ 1150 4700
+NoConn ~ 1150 4800
+NoConn ~ 1150 4900
+NoConn ~ 1150 5000
+NoConn ~ 1150 5400
 $EndSCHEMATC

Commit message: e
Parts:
- added 3.3v: Conn_01x02, symbol Connector_Generic:Conn_01x02
- gave numbers to parts that had none: 1
Connections:
- net +3V3: now also 3.3v.1 (Pin_1)
- net GND: now also 3.3v.2 (Pin_2)
- net PWM-0 renamed PWM_0
- net PWM-1 renamed PWM_1
- net PWM-2 renamed PWM_2
- net PWM-3 renamed PWM_3
- net PWM-4 renamed PWM_4
- net PWM-5 renamed PWM_5
- net PWM-6 renamed PWM_6
- net PWM-7 renamed PWM_7
- net PWM-8 renamed PWM_8
Other:
- moved on the sheet: I2C

Commit message: Board Prototrype
e
Parts:
- added R1, R2: R, Resistor_SMD:R_0805_2012Metric_Pad1.15x1.40mm_HandSolder, symbol Device:R
- 3.3v1: renamed from 3.3v; footprint (none) -> 2.54mm_Pin_Headers:PinHeader_1x02_P2.54mm_Vertical
- CBConn1: renamed from CBConn; footprint (none) -> 2.54mm_Pin_Headers:PinHeader_1x02_P2.54mm_Vertical
- I2C1, I2C2: renamed from I2C; footprint (none) -> 2.54mm_Pin_Headers:PinHeader_1x04_P2.54mm_Vertical
- J1: renamed from J?; footprint (none) -> 2.54mm_Pin_Headers:PinHeader_1x02_P2.54mm_Vertical
- PWM-0, PWM-1, PWM-10, PWM-11, PWM-2, PWM-3, PWM-4, PWM-5, PWM-6, PWM-7, PWM-8, PWM-9: footprint (none) -> 2.54mm_Pin_Headers:PinHeader_1x03_P2.54mm_Vertical
- PWM-12, PWM-13, PWM-14: renamed from PWM-?; footprint (none) -> 2.54mm_Pin_Headers:PinHeader_1x03_P2.54mm_Vertical
- XT-60: footprint (none) -> Arduino Project:XT60
Connections:
- net +3V3: now also R1.1, R2.1
- net I2C_SCL: now also R1.2
- net I2C_SDA: now also R2.2
- net PWM_13: now also U1.21 (29_PWM_CAN0TX_Touch); no longer U1.47 (20_A6_PWM_CS0_SCK1)
- net PWM_14: now also U1.22 (30_PWM_CAN0RX_Touch); no longer U1.48 (21_A7_PWM_CS0_MOSI1)
- net PWM_6: now also U1.48 (21_A7_PWM_CS0_MOSI1); no longer U1.21 (29_PWM_CAN0TX_Touch)
- net PWM_7: now also U1.47 (20_A6_PWM_CS0_SCK1); no longer U1.22 (30_PWM_CAN0RX_Touch)
- net PWM_8: now also U1.35 (38_A19_PWM_SDA1); no longer U1.32 (35_A16_PWM)
- net PWM-10 renamed PWM_10
- net PWM_10: now also U1.33 (36_A17_PWM); no longer U1.34 (37_A18_PWM_SCL1)
- net PWM-11 renamed PWM_11
- net PWM_11: now also U1.32 (35_A16_PWM); no longer U1.35 (38_A19_PWM_SDA1)
- net PWM-9 renamed PWM_9
- net PWM_9: now also U1.34 (37_A18_PWM_SCL1); no longer U1.33 (36_A17_PWM)
