File: Arduino Project/Arduino Project.sch (KiCad schematic (older format))
At the start: 26 parts, among them J1 Conn_01x02, U1 Teensy3.5

Commit message: Final Board
Parts:
- gave numbers to parts that had none: 2
Connections:
- net PWM_10: now also U1.22 (30_PWM_CAN0RX_Touch); no longer U1.33 (36_A17_PWM)
- net PWM_11: now also U1.41 (14_A0_PWM_SCK0); no longer U1.32 (35_A16_PWM)
- net PWM_12: now also U1.34 (37_A18_PWM_SCL1); no longer U1.41 (14_A0_PWM_SCK0)
- net PWM_13: now also U1.33 (36_A17_PWM); no longer U1.21 (29_PWM_CAN0TX_Touch)
- net PWM_14: now also U1.32 (35_A16_PWM); no longer U1.22 (30_PWM_CAN0RX_Touch)
- net PWM_9: now also U1.21 (29_PWM_CAN0TX_Touch); no longer U1.34 (37_A18_PWM_SCL1)
Changed lines of the file:
@@
 Text GLabel 1150 4500 0    50   Input ~ 0
 PWM_8
-Text GLabel 1150 4300 0    50   Input ~ 0
+Text GLabel 1150 3200 0    50   Input ~ 0
 PWM_10
 $Comp
@@
 Text GLabel 8650 4800 0    50   Input ~ 0
 PWM_13
-Text GLabel 1150 5100 0    50   Input ~ 0
+Text GLabel 1150 4400 0    50   Input ~ 0
 PWM_12
 $Comp
@@
 	0    1    1    0
 $EndComp
-Text GLabel 1150 3100 0    50   Input ~ 0
+Text GLabel 1150 4300 0    50   Input ~ 0
 PWM_13
-Text GLabel 1150 3200 0    50   Input ~ 0
+Text GLabel 1150 4200 0    50   Input ~ 0
 PWM_14
 Text GLabel 1150 5200 0    50   Input ~ 0
@@
 Text GLabel 9750 2850 0    50   Input ~ 0
 PWM_8
-Text GLabel 1150 4400 0    50   Input ~ 0
+Text GLabel 1150 3100 0    50   Input ~ 0
 PWM_9
 Text GLabel 9750 3850 0    50   Input ~ 0
 PWM_10
-Text GLabel 1150 4200 0    50   Input ~ 0
+Text GLabel 1150 5100 0    50   Input ~ 0
 PWM_11
 $Comp
@@
 $EndComp
 $Comp
-L Isolator:NSL-32 U?
+L Isolator:NSL-32 U2
 U 1 1 5D9E88FE
 P 5450 4050
-F 0 "U?" H 5450 4367 50  0000 C CNN
+F 0 "U2" H 5450 4367 50  0000 C CNN
 F 1 "NSL-32" H 5450 4276 50  0000 C CNN
 F 2 "OptoDevice:Luna_NSL-32" H 5450 3750 50  0001 C CNN
@@
 $EndComp
 $Comp
-L Device:R R?
+L Device:R R3
 U 1 1 5D9E8965
 P 5000 3950
-F 0 "R?" V 4793 3950 50  0000 C CNN
+F 0 "R3" V 4793 3950 50  0000 C CNN
 F 1 "R" V 4884 3950 50  0000 C CNN
 F 2 "" V 4930 3950 50  0001 C CNN
@@
 CBEnable
 $Comp
-L power:GND #PWR?
+L power:GND #PWR0135
 U 1 1 5D9E946E
 P 5150 4150
-F 0 "#PWR?" H 5150 3900 50  0001 C CNN
+F 0 "#PWR0135" H 5150 3900 50  0001 C CNN
 F 1 "GND" V 5155 4022 50  0000 R CNN
 F 2 "" H 5150 4150 50  0001 C CNN
@@
 CBEnable_5v
 $Comp
-L power:+5V #PWR?
+L power:+5V #PWR0136
 U 1 1 5D9E958C
 P 5750 3950
-F 0 "#PWR?" H 5750 3800 50  0001 C CNN
+F 0 "#PWR0136" H 5750 3800 50  0001 C CNN
 F 1 "+5V" V 5765 4078 50  0000 L CNN
 F 2 "" H 5750 3950 50  0001 C CNN

Commit message: final
Parts:
- renumbered J1 to Switch1
Changed lines of the file:
@@
 I2C_SDA
 $Comp
-L Connector_Generic:Conn_01x02 J1
+L Connector_Generic:Conn_01x02 Switch1
 U 1 1 5D95555F
 P 10050 1250
-F 0 "J1" H 10130 1242 50  0000 L CNN
+F 0 "Switch1" H 10130 1242 50  0000 L CNN
 F 1 "Conn_01x02" H 10130 1151 50  0000 L CNN
 F 2 "2.54mm_Pin_Headers:PinHeader_1x02_P2.54mm_Vertical" H 10050 1250 50  0001 C CNN
