File: Arduino Project/Arduino Project.kicad_pcb (KiCad board)
At the start: 2 copper layers, 92 x 45 mm, 24 parts, among them J1 Conn_01x02, U1 Teensy3.5

Commit message: Final Board
Parts:
- added R3: R, Resistor_SMD:R_0805_2012Metric_Pad1.15x1.40mm_HandSolder, F.Cu at (158.5, 59.0)
- added U2: NSL-32, Package_SO:SOP-4_3.8x4.1mm_P2.54mm, F.Cu at (156.5, 53.5)
Connections:
- CBConn1 pad 1: CBEnable -> CBEnable_5v
- U1 pad 21: PWM_13 -> PWM_9
- U1 pad 22: PWM_14 -> PWM_10
- U1 pad 32: PWM_11 -> PWM_14
- U1 pad 33: PWM_10 -> PWM_13
- U1 pad 34: PWM_9 -> PWM_12
- U1 pad 41: PWM_12 -> PWM_11
Routing:
- net CBEnable_5v: track 0.00 -> 33.4 mm
- net CBEnable: track 14.4 -> 47.3 mm
- net PWM_9: track 46.4 -> 18.4 mm
- net +5V: track 90.2 -> 115.1 mm
- net PWM_10: track 43.3 -> 21.3 mm
- net PWM_12: track 73.6 -> 51.8 mm
- net PWM_11: track 46.0 -> 61.1 mm
- net GND: track 0.00 -> 13.2 mm
- net PWM_13: track 39.1 -> 51.7 mm
- net PWM_14: track 43.8 -> 52.9 mm
- net Net-(R3-Pad1): track 0.00 -> 4.34 mm

Commit message: Final v2
e
Routing:
- net +5V: track 115.1 -> 115.9 mm
Other:
- net class 5v added: clearance 0.2, trace_width 0.4, via_dia 0.8, via_drill 0.4
Changed lines of the file:
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@@
     (uvia_drill 0.1)
     (add_net +3V3)
-    (add_net +5V)
     (add_net CBEnable)
-    (add_net CBEnable_5v)
-    (add_net GND)
     (add_net I2C_SCL)
     (add_net I2C_SDA)
@@
     (add_net PWM_9)
     (add_net Saftey_Switch)
+  )
+  (net_class 5v ""
+    (clearance 0.2)
+    (trace_width 0.4)
+    (via_dia 0.8)
+    (via_drill 0.4)
+    (uvia_dia 0.3)
+    (uvia_drill 0.1)
+    (add_net +5V)
+    (add_net CBEnable_5v)
+    (add_net GND)
   )
   (module Package_SO:SOP-4_3.8x4.1mm_P2.54mm (layer F.Cu)
@@
   (segment (start 137.5 48.5) (end 139 47) (width 0.25) (layer B.Cu) (net 1))
   (segment (start 105 46) (end 105 48.5) (width 0.25) (layer B.Cu) (net 1) (status 400000))
-  (segment (start 159.25 52.23) (end 159.25 47.25) (width 0.25) (layer F.Cu) (net 2) (status 400000))
-  (segment (start 158 46) (end 151.54 46) (width 0.25) (layer F.Cu) (net 2) (status 800000))
-  (segment (start 159.25 47.25) (end 158 46) (width 0.25) (layer F.Cu) (net 2))
+  (segment (start 159.25 52.23) (end 159.25 47.75) (width 0.4) (layer F.Cu) (net 2) (status 400000))
+  (segment (start 157.5 46) (end 151.54 46) (width 0.4) (layer F.Cu) (net 2) (status 800000))
+  (segment (start 159.25 47.75) (end 157.5 46) (width 0.4) (layer F.Cu) (net 2))
   (segment (start 157.475 59) (end 153 59) (width 0.25) (layer F.Cu) (net 3) (status 400000))
   (segment (start 118.900002 51) (end 116.555001 53.345001) (width 0.25) (layer F.Cu) (net 3) (status 800000))
@@
   (segment (start 134.335001 63.505001) (end 168.505001 63.505001) (width 0.25) (layer B.Cu) (net 41) (status C00000))
   (segment (start 168.505001 63.505001) (end 169 64) (width 0.25) (layer B.Cu) (net 41) (status C00000))
-  (segment (start 153.75 54.77) (end 153.75 54.25) (width 0.25) (layer F.Cu) (net 41) (status 400000))
-  (segment (start 165.5 64) (end 169 64) (width 0.25) (layer F.Cu) (net 41) (status 800000))
-  (segment (start 164 62.5) (end 165.5 64) (width 0.25) (layer F.Cu) (net 41))
-  (segment (start 164 55) (end 164 62.5) (width 0.25) (layer F.Cu) (net 41))
-  (segment (start 162.5 53.5) (end 164 55) (width 0.25) (layer F.Cu) (net 41))
-  (segment (start 154.5 53.5) (end 162.5 53.5) (width 0.25) (layer F.Cu) (net 41))
-  (segment (start 153.75 54.25) (end 154.5 53.5) (width 0.25) (layer F.Cu) (net 41))
-  (segment (start 125 46) (end 125 48.5) (width 0.25) (layer F.Cu) (net 72) (status 400000))
-  (segment (start 153.75 51.25) (end 153.75 52.23) (width 0.25) (layer F.Cu) (net 72) (status 800000))
-  (segment (start 152.5 50) (end 153.75 51.25) (width 0.25) (layer F.Cu) (net 72))
-  (segment (start 126.5 50) (end 152.5 50) (width 0.25) (layer F.Cu) (net 72))
-  (segment (start 125 48.5) (end 126.5 50) (width 0.25) (layer F.Cu) (net 72))
+  (segment (start 153.75 54.77) (end 153.75 53.75) (width 0.4) (layer F.Cu) (net 41) (status 400000))
+  (segment (start 164 64) (end 169 64) (width 0.4) (layer F.Cu) (net 41) (status 800000))
+  (segment (start 162.5 62.5) (end 164 64) (width 0.4) (layer F.Cu) (net 41))
+  (segment (start 162.5 54) (end 162.5 62.5) (width 0.4) (layer F.Cu) (net 41))
+  (segment (start 162 53.5) (end 162.5 54) (width 0.4) (layer F.Cu) (net 41))
+  (segment (start 154 53.5) (end 162 53.5) (width 0.4) (layer F.Cu) (net 41))
+  (segment (start 153.75 53.75) (end 154 53.5) (width 0.4) (layer F.Cu) (net 41))
+  (segment (start 153.75 52.23) (end 153.75 51.25) (width 0.4) (layer F.Cu) (net 72) (status 400000))
+  (segment (start 125 48.5) (end 125 46) (width 0.4) (layer F.Cu) (net 72) (status 800000))
+  (segment (start 126.5 50) (end 125 48.5) (width 0.4) (layer F.Cu) (net 72))
+  (segment (start 152.5 50) (end 126.5 50) (width 0.4) (layer F.Cu) (net 72))
+  (segment (start 153.75 51.25) (end 152.5 50) (width 0.4) (layer F.Cu) (net 72))
   (segment (start 159.525 59) (end 159.525 55.045) (width 0.25) (layer F.Cu) (net 73) (status C00000))
   (segment (start 159.525 55.045) (end 159.25 54.77) (width 0.25) (layer F.Cu) (net 73) (status C00000))

Commit message: final
Parts:
- removed J1: Conn_01x02, 2.54mm_Pin_Headers:PinHeader_1x02_P2.54mm_Vertical
- added SW: Conn_01x02, 2.54mm_Pin_Headers:PinHeader_1x02_P2.54mm_Vertical, F.Cu at (139.0, 46.0)
- renumbered 3.3v1 to 3.3V_OP, XT-60 to 5V_IN, PWM-0 to PWM0, PWM-1 to PWM1, PWM-10 to PWM10, PWM-11 to PWM11, PWM-12 to PWM12, PWM-13 to PWM13, PWM-14 to PWM14, PWM-2 to PWM2, PWM-3 to PWM3, PWM-4 to PWM4, PWM-5 to PWM5, PWM-6 to PWM6, PWM-7 to PWM7, PWM-8 to PWM8, PWM-9 to PWM9, CBConn1 to SW_PWR
Routing:
- net I2C_SDA: track 27.0 -> 29.8 mm, vias 2 -> 0
- net PWM_7: track 48.9 -> 49.9 mm
- net PWM_6: track 48.9 -> 48.3 mm
Other:
- board text added: "Teensy PWM & I2C ASUR 2020"
- board text removed: "Teensy PWM & I2C BY ASUR"
